File: kicad/LEDCube8х16/LEDCube_8x16.sch (KiCad schematic (older format))
At the start: 60 parts, among them J1 USB_OTG, J10 6, J11 7, J12 8, J13 RX, J14 TX, J3 1, J4 2, J5 3, J6 vert layers, J7 ICSP, J8 4, J9 5, Q1 BCP 51.115, Q10 BCP 51.115, Q11 BCP 51.115, Q12 BCP 51.115, Q13 BCP 51.115, Q14 BCP 51.115, Q15 BCP 51.115, Q16 BCP 51.115, Q2 BCP 51.115, Q3 BCP 51.115, Q4 BCP 51.115, Q5 BCP 51.115, Q6 BCP 51.115, Q7 BCP 51.115, Q8 BCP 51.115, Q9 BCP 51.115, U1 ATMEGA644P, U2 TSOP312xx, Y1 16mhz

Commit message: fixes in scheme
Parts:
- added C4: 4400 mkf x 6.3 v, Capacitors_THT:CP_Radial_D18.0mm_P7.50mm, symbol CP
Connections:
- net GND: now also C4.2
- net at J1.1 (VBUS), J7.4 (P4), MB1.24 (VDD)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: now also C4.1
Changed lines of the file:
@@
 EESchema Schematic File Version 2
+LIBS:74xgxx
+LIBS:74xx
+LIBS:ac-dc
+LIBS:actel
+LIBS:adc-dac
+LIBS:allegro
+LIBS:Altera
+LIBS:analog_devices
+LIBS:analog_switches
+LIBS:atmel
+LIBS:audio
+LIBS:battery_management
+LIBS:bbd
+LIBS:bosch
+LIBS:brooktre
+LIBS:cmos_ieee
+LIBS:cmos4000
+LIBS:conn
+LIBS:contrib
+LIBS:cypress
+LIBS:dc-dc
+LIBS:device
+LIBS:digital-audio
+LIBS:diode
+LIBS:display
+LIBS:dsp
+LIBS:elec-unifil
+LIBS:ESD_Protection
+LIBS:ftdi
+LIBS:gennum
+LIBS:graphic
+LIBS:hc11
+LIBS:intel
+LIBS:interface
+LIBS:ir
+LIBS:Lattice
+LIBS:leds
+LIBS:linear
+LIBS:logo
+LIBS:maxim
+LIBS:mechanical
+LIBS:memory
+LIBS:microchip
+LIBS:microchip_dspic33dsc
+LIBS:microchip_pic10mcu
+LIBS:microchip_pic12mcu
+LIBS:microchip_pic16mcu
+LIBS:microchip_pic18mcu
+LIBS:microchip_pic24mcu
+LIBS:microchip_pic32mcu
+LIBS:microcontrollers
+LIBS:modules
+LIBS:motor_drivers
+LIBS:motorola
+LIBS:motors
+LIBS:msp430
+LIBS:nordicsemi
+LIBS:nxp
+LIBS:nxp_armmcu
+LIBS:onsemi
+LIBS:opto
+LIBS:Oscillators
+LIBS:philips
 LIBS:power
-LIBS:device
+LIBS:Power_Management
+LIBS:powerint
+LIBS:pspice
+LIBS:references
+LIBS:regul
+LIBS:relays
+LIBS:rfcom
+LIBS:sensors
+LIBS:silabs
+LIBS:siliconi
+LIBS:stm8
+LIBS:stm32
+LIBS:supertex
+LIBS:switches
+LIBS:texas
+LIBS:transf
 LIBS:transistors
-LIBS:conn
-LIBS:linear
-LIBS:regul
-LIBS:74xx
-LIBS:cmos4000
-LIBS:adc-dac
-LIBS:memory
+LIBS:triac_thyristor
+LIBS:ttl_ieee
+LIBS:valves
+LIBS:video
+LIBS:wiznet
+LIBS:Worldsemi
+LIBS:Xicor
 LIBS:xilinx
-LIBS:microcontrollers
-LIBS:dsp
-LIBS:microchip
-LIBS:analog_switches
-LIBS:motorola
-LIBS:texas
-LIBS:intel
-LIBS:audio
-LIBS:interface
-LIBS:digital-audio
-LIBS:philips
-LIBS:display
-LIBS:cypress
-LIBS:siliconi
-LIBS:opto
-LIBS:atmel
-LIBS:contrib
-LIBS:valves
+LIBS:zetex
+LIBS:Zilog
 LIBS:MY
 LIBS:LEDCube_8x16-cache
@@
 	2450 4500 2150 4500
 Wire Wire Line
-	1750 6600 3400 6600
+	1750 6600 3600 6600
 Connection ~ 3400 6600
 Wire Wire Line
@@
 Wire Wire Line
 	15100 5450 15100 2450
+$Comp
+L CP C4
+U 1 1 61B07822
+P 3750 6600
+F 0 "C4" H 3775 6700 50  0000 L CNN
+F 1 "4400 mkf x 6.3 v" H 3775 6500 50  0000 L CNN
+F 2 "Capacitors_THT:CP_Radial_D18.0mm_P7.50mm" H 3788 6450 50  0001 C CNN
+F 3 "" H 3750 6600 50  0001 C CNN
+	1    3750 6600
+	0    -1   -1   0
+$EndComp
+$Comp
+L GND #PWR014
+U 1 1 61B07A42
+P 4100 6700
+F 0 "#PWR014" H 4100 6450 50  0001 C CNN
+F 1 "GND" H 4100 6550 50  0000 C CNN
+F 2 "" H 4100 6700 50  0001 C CNN
+F 3 "" H 4100 6700 50  0001 C CNN
+	1    4100 6700
+	1    0    0    -1
+$EndComp
+Wire Wire Line
+	3900 6600 4100 6600
+Wire Wire Line
+	4100 6600 4100 6700
 $EndSCHEMATC

Commit message: added resistor between mcu and leds
Parts:
- added R22: 4R, Resistors_THT:R_Axial_DIN0411_L9.9mm_D3.6mm_P7.62mm_Vertical, symbol R
- R1, R3, R4, R5: value R -> 1k
Connections:
- net at MB1.24 (VDD), MB2.24 (VDD), MB3.24 (VDD)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: now also R22.2; no longer C4.1, J1.1 (VBUS), J7.4 (P4), R2.2, U1.17 (VCC), U1.27 (VCC), U1.38 (vcc), U1.5 (VCC), U2.2 (Vs)
- new net: C4.1, J1.1 (VBUS), J7.4 (P4), R2.2, R22.1, U1.17 (VCC), U1.27 (VCC), U1.38 (vcc), U1.5 (VCC), U2.2 (Vs)
Changed lines of the file:
@@
 P 12100 8750
 F 0 "R5" V 12180 8750 50  0000 C CNN
-F 1 "R" V 12100 8750 50  0000 C CNN
+F 1 "1k" V 12100 8750 50  0000 C CNN
 F 2 "Resistors_SMD:R_0805" V 12030 8750 50  0001 C CNN
 F 3 "" H 12100 8750 50  0001 C CNN
@@
 P 9000 8750
 F 0 "R4" V 9080 8750 50  0000 C CNN
-F 1 "R" V 9000 8750 50  0000 C CNN
+F 1 "1k" V 9000 8750 50  0000 C CNN
 F 2 "Resistors_SMD:R_0805" V 8930 8750 50  0001 C CNN
 F 3 "" H 9000 8750 50  0001 C CNN
@@
 P 5950 8800
 F 0 "R3" V 6030 8800 50  0000 C CNN
-F 1 "R" V 5950 8800 50  0000 C CNN
+F 1 "1k" V 5950 8800 50  0000 C CNN
 F 2 "Resistors_SMD:R_0805" V 5880 8800 50  0001 C CNN
 F 3 "" H 5950 8800 50  0001 C CNN
@@
 P 2950 8800
 F 0 "R1" V 3030 8800 50  0000 C CNN
-F 1 "R" V 2950 8800 50  0000 C CNN
+F 1 "1k" V 2950 8800 50  0000 C CNN
 F 2 "Resistors_SMD:R_0805" V 2880 8800 50  0001 C CNN
 F 3 "" H 2950 8800 50  0001 C CNN
@@
 Connection ~ 1700 3950
 Wire Wire Line
-	3400 5150 3400 8450
+	3400 5150 3400 7050
 Wire Wire Line
 	1300 8000 1300 9000
@@
 Wire Wire Line
 	4700 3700 4700 2950
-Wire Wire Line
-	3500 2100 3500 3250
-Wire Wire Line
-	3500 2950 1400 2950
 Wire Wire Line
 	1400 2950 1400 3850
@@
 	15500 2100 15500 2000
 Wire Wire Line
-	3500 2100 15500 2100
-Wire Wire Line
-	4800 2100 4800 2000
-Connection ~ 3500 2950
+	4800 2100 15500 2100
+Wire Wire Line
+	4800 8450 4800 2000
 Connection ~ 4800 2100
 Wire Wire Line
@@
 Wire Wire Line
 	4100 6600 4100 6700
+Wire Wire Line
+	3500 2950 1400 2950
+Wire Wire Line
+	3500 2950 3500 3250
+Connection ~ 4800 8450
+$Comp
+L R R22
+U 1 1 61B0ECF9
+P 3400 7200
+F 0 "R22" V 3480 7200 50  0000 C CNN
+F 1 "4R" V 3400 7200 50  0000 C CNN
+F 2 "Resistors_THT:R_Axial_DIN0411_L9.9mm_D3.6mm_P7.62mm_Vertical" V 3330 7200 50  0001 C CNN
+F 3 "" H 3400 7200 50  0001 C CNN
+	1    3400 7200
+	1    0    0    -1
+$EndComp
+Wire Wire Line
+	3400 7350 3400 8450
 $EndSCHEMATC
